Commit message: Reorganize retargeting package and offline benchmarks

File: ws_ros2/src/my_robot_description/urdf/leap_hand/leap_hand_paxini.urdf.xacro (robot description, xacro)
@@ -1,5 +1,5 @@
 <?xml version="1.0"?>
 <robot xmlns:xacro="http://www.ros.org/wiki/xacro">
-    <xacro:macro name="leap_hand_custom_tac3d" params="mesh_dir">
+    <xacro:macro name="leap_hand_paxini" params="mesh_dir">
         <xacro:include
             filename="$(find my_robot_description)/urdf/leap_hand/leap_hand_body.urdf.xacro" />

File: ws_ros2/src/my_robot_description/urdf/panda.xacro (robot description, xacro)
@@ -1,4 +1,4 @@
 <?xml version="1.0"?>
-<robot name="panda_leap_tac3d" xmlns:xacro="http://www.ros.org/wiki/xacro">
+<robot name="panda" xmlns:xacro="http://www.ros.org/wiki/xacro">
     <xacro:arg name="panda_mesh_dir" default="./panda/meshes/" />
     <xacro:include

File: ws_ros2/src/my_robot_description/urdf/panda_leap_paxini.xacro (robot description, xacro)
@@ -1,4 +1,4 @@
 <?xml version="1.0"?>
-<robot name="panda_leap_tac3d" xmlns:xacro="http://www.ros.org/wiki/xacro">
+<robot name="panda_leap_paxini" xmlns:xacro="http://www.ros.org/wiki/xacro">
     <xacro:arg name="panda_mesh_dir" default="./panda/meshes/" />
     <xacro:arg name="leap_mesh_dir" default="./leap_hand/meshes/" />
@@ -8,5 +8,5 @@
     <xacro:include
         filename="$(find my_robot_description)/urdf/leap_hand/leap_hand_paxini.urdf.xacro" />
-    <xacro:leap_hand_custom_tac3d mesh_dir="$(arg leap_mesh_dir)" />
+    <xacro:leap_hand_paxini mesh_dir="$(arg leap_mesh_dir)" />
     <joint name="panda_leap" type="fixed">
         <origin
