Commit message: feat: add headless MuJoCo retargeting workflows

File: assets/robots/panda_leap_paxini/urdf/panda_leap_paxini.urdf (robot description, URDF)
Before this commit: robot panda_leap_paxini, 44 links, 43 joints
Links:
- link dip: geometry collision mesh filename=../meshes/leap_hand/dip.stl; visual mesh filename=../meshes/leap_hand/dip.stl
- link dip_2: geometry collision mesh filename=../meshes/leap_hand/dip.stl; visual mesh filename=../meshes/leap_hand/dip.stl
- link dip_3: geometry collision mesh filename=../meshes/leap_hand/dip.stl; visual mesh filename=../meshes/leap_hand/dip.stl
- link fingertip: geometry collision mesh filename=../meshes/leap_hand/fingertip_base.stl; visual mesh filename=../meshes/leap_hand/fingertip_base.stl
- link fingertip_2: geometry collision mesh filename=../meshes/leap_hand/fingertip_base.stl; visual mesh filename=../meshes/leap_hand/fingertip_base.stl
- link fingertip_2_new: geometry collision mesh filename=../meshes/leap_hand/paxini_base.STL scale=0.001 0.001 0.001; visual mesh filename=../meshes/leap_hand/paxini_base.STL scale=0.001 0.001 0.001
- link fingertip_2_new_tip: geometry collision mesh filename=../meshes/leap_hand/paxini_fingertip.STL scale=1 1 1; visual mesh filename=../meshes/leap_hand/paxini_fingertip.STL scale=1 1 1
- link fingertip_3: geometry collision mesh filename=../meshes/leap_hand/fingertip_base.stl; visual mesh filename=../meshes/leap_hand/fingertip_base.stl
- link fingertip_3_new: geometry collision mesh filename=../meshes/leap_hand/paxini_base.STL scale=0.001 0.001 0.001; visual mesh filename=../meshes/leap_hand/paxini_base.STL scale=0.001 0.001 0.001
- link fingertip_3_new_tip: geometry collision mesh filename=../meshes/leap_hand/paxini_fingertip.STL scale=1 1 1; visual mesh filename=../meshes/leap_hand/paxini_fingertip.STL scale=1 1 1
- link fingertip_new: geometry collision mesh filename=../meshes/leap_hand/paxini_base.STL scale=0.001 0.001 0.001; visual mesh filename=../meshes/leap_hand/paxini_base.STL scale=0.001 0.001 0.001
- link fingertip_new_tip: geometry collision mesh filename=../meshes/leap_hand/paxini_fingertip.STL scale=1 1 1; visual mesh filename=../meshes/leap_hand/paxini_fingertip.STL scale=1 1 1
- link mcp_joint: geometry collision mesh filename=../meshes/leap_hand/mcp_joint.stl; visual mesh filename=../meshes/leap_hand/mcp_joint.stl
- link mcp_joint_2: geometry collision mesh filename=../meshes/leap_hand/mcp_joint.stl; visual mesh filename=../meshes/leap_hand/mcp_joint.stl
- link mcp_joint_3: geometry collision mesh filename=../meshes/leap_hand/mcp_joint.stl; visual mesh filename=../meshes/leap_hand/mcp_joint.stl
- link palm_lower: geometry collision mesh filename=../meshes/leap_hand/palm_lower.stl; visual mesh filename=../meshes/leap_hand/palm_lower.stl
- link panda_link0: geometry collision mesh filename=../meshes/panda/collision/link0.obj; visual mesh filename=../meshes/panda/visual/link0.stl
- link panda_link1: geometry collision mesh filename=../meshes/panda/collision/link1.obj; visual mesh filename=../meshes/panda/visual/link1.stl
- link panda_link2: geometry collision mesh filename=../meshes/panda/collision/link2.obj; visual mesh filename=../meshes/panda/visual/link2.stl
- link panda_link3: geometry collision mesh filename=../meshes/panda/collision/link3.obj; visual mesh filename=../meshes/panda/visual/link3.stl
- link panda_link4: geometry collision mesh filename=../meshes/panda/collision/link4.obj; visual mesh filename=../meshes/panda/visual/link4.stl
- link panda_link5: geometry collision mesh filename=../meshes/panda/collision/link5.obj; visual mesh filename=../meshes/panda/visual/link5.stl
- link panda_link6: geometry collision mesh filename=../meshes/panda/collision/link6.obj; visual mesh filename=../meshes/panda/visual/link6.stl
- link panda_link7: geometry collision mesh filename=../meshes/panda/collision/link7.obj; visual mesh filename=../meshes/panda/visual/link7.stl
- link pip: geometry collision mesh filename=../meshes/leap_hand/pip.stl; visual mesh filename=../meshes/leap_hand/pip.stl
- link pip_2: geometry collision mesh filename=../meshes/leap_hand/pip.stl; visual mesh filename=../meshes/leap_hand/pip.stl
- link pip_3: geometry collision mesh filename=../meshes/leap_hand/pip.stl; visual mesh filename=../meshes/leap_hand/pip.stl
- link pip_4: geometry collision mesh filename=../meshes/leap_hand/pip.stl; visual mesh filename=../meshes/leap_hand/pip.stl
- link thumb_dip: geometry collision mesh filename=../meshes/leap_hand/thumb_dip.stl; visual mesh filename=../meshes/leap_hand/thumb_dip.stl
- link thumb_fingertip: geometry collision mesh filename=../meshes/leap_hand/thumb_fingertip_base.stl; visual mesh filename=../meshes/leap_hand/thumb_fingertip_base.stl
- link thumb_fingertip_new: geometry collision mesh filename=../meshes/leap_hand/paxini_base.STL scale=0.001 0.001 0.001; visual mesh filename=../meshes/leap_hand/paxini_base.STL scale=0.001 0.001 0.001
- link thumb_fingertip_new_tip: geometry collision mesh filename=../meshes/leap_hand/paxini_fingertip.STL scale=1 1 1; visual mesh filename=../meshes/leap_hand/paxini_fingertip.STL scale=1 1 1
- link thumb_pip: geometry collision mesh filename=../meshes/leap_hand/thumb_pip.stl; visual mesh filename=../meshes/leap_hand/thumb_pip.stl
